File: gadgeteer_HD44780.brd (EAGLE design)
At the start: 42 x 19 mm, 9 parts, among them T1 3904

Commit message: [FIX] Changed C1 to 1206K (Kemet) metric size
Parts:
- removed C2: 4.7uF, adafruit:C1206
- added C1: 4.7uF, adafruit:C1206K
- S1: value (none) -> 5K
- renumbered R25 to R2
Connections:
- net GND: now also C1.2; no longer C2.2
- net N$2: now also C1.1; no longer C2.1
Changed lines of the file:
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@@
 <grid distance="0.125" unitdist="mm" unit="mm" style="lines" multiple="1" display="yes" altdistance="0.025" altunitdist="inch" altunit="inch"/>
 <layers>
-<layer number="1" name="Top" color="4" fill="1" visible="no" active="yes"/>
+<layer number="1" name="Top" color="4" fill="1" visible="yes" active="yes"/>
 <layer number="2" name="Route2" color="1" fill="3" visible="no" active="no"/>
 <layer number="3" name="Route3" color="4" fill="3" visible="no" active="no"/>
 <layer number="14" name="Route14" color="1" fill="6" visible="no" active="no"/>
 <layer number="15" name="Route15" color="4" fill="6" visible="no" active="no"/>
-<layer number="16" name="Bottom" color="1" fill="1" visible="no" active="yes"/>
+<layer number="16" name="Bottom" color="1" fill="1" visible="yes" active="yes"/>
 <layer number="17" name="Pads" color="2" fill="1" visible="yes" active="yes"/>
 <layer number="18" name="Vias" color="2" fill="1" visible="yes" active="yes"/>
@@
 <attribute name="VALUE" x="41.27" y="19.81" size="1.27" layer="27" rot="R180"/>
 </element>
-<element name="C2" library="adafruit" package="C1206" value="4.7uF" x="31.5" y="4" rot="R270"/>
-<element name="R25" library="adafruit" package="R0603" value="330" x="10" y="3" smashed="yes" rot="R180">
+<element name="R2" library="adafruit" package="R0603" value="330" x="10" y="3" smashed="yes" rot="R180">
 <attribute name="NAME" x="12" y="4.5" size="1.27" layer="25" rot="R270"/>
 <attribute name="VALUE" x="10.889" y="5.032" size="1.27" layer="27" rot="R180"/>
@@
 <element name="U$2" library="Gadgeteer" package="HOLE3.2" value="" x="4" y="4"/>
 <element name="U$3" library="Gadgeteer" package="HOLE3.2" value="" x="38" y="4"/>
-<element name="S1" library="adafruit" package="EG1218" value="" x="21" y="11" smashed="yes"/>
+<element name="S1" library="adafruit" package="EG1218" value="5K" x="21" y="11" smashed="yes"/>
+<element name="C1" library="adafruit" package="C1206K" value="4.7uF" x="31.375" y="4.25" rot="R270"/>
 </elements>
 <signals>
@@
 <contactref element="JP1" pad="1"/>
 <contactref element="JP1" pad="5"/>
-<contactref element="C2" pad="2"/>
 <contactref element="T1" pad="E"/>
 <contactref element="Y" pad="10"/>
@@
 <wire x1="29.5" y1="5" x2="31.5" y2="3" width="0.254" layer="1"/>
 <wire x1="29.5" y1="16" x2="29.5" y2="5" width="0.254" layer="1"/>
-<wire x1="31.5" y1="3" x2="31.5" y2="2.6" width="0.254" layer="1"/>
 <wire x1="29.5" y1="16" x2="29.84" y2="16" width="0.254" layer="1"/>
 <wire x1="39" y1="15" x2="40" y2="16" width="0.254" layer="1"/>
 <wire x1="39" y1="10" x2="39" y2="15" width="0.254" layer="1"/>
 <wire x1="31.5" y1="2.5" x2="39" y2="10" width="0.254" layer="1"/>
-<wire x1="31.5" y1="2.5" x2="31.5" y2="2.6" width="0.254" layer="1"/>
 <wire x1="18.5" y1="3.5" x2="17" y2="2" width="0.254" layer="16"/>
 <wire x1="32.5" y1="3.5" x2="18.5" y2="3.5" width="0.254" layer="16"/>
@@
 <wire x1="40" y1="16" x2="40" y2="11" width="0.254" layer="16"/>
 <via x="17" y="2" extent="1-16" drill="0.6096"/>
+<contactref element="C1" pad="2"/>
+<wire x1="31.5" y1="3" x2="31.375" y2="2.75" width="0.1524" layer="1"/>
+<wire x1="31.5" y1="2.5" x2="31.375" y2="2.75" width="0.1524" layer="1"/>
 </signal>
 <signal name="+5V">
@@
 <contactref element="JP1" pad="15"/>
 <contactref element="JP1" pad="2"/>
-<contactref element="C2" pad="1"/>
 <contactref element="S1" pad="P"/>
-<wire x1="31.5" y1="7.5" x2="31.5" y2="5.5" width="0.254" layer="1"/>
+<wire x1="31.5" y1="7.5" x2="31.5" y2="6" width="0.254" layer="1"/>
+<wire x1="31.5" y1="6" x2="31.5" y2="5.5" width="0.254" layer="1"/>
 <wire x1="37" y1="13" x2="31.5" y2="7.5" width="0.254" layer="16"/>
 <wire x1="37" y1="16" x2="37" y2="13" width="0.254" layer="16"/>
-<wire x1="31.5" y1="5.5" x2="31.5" y2="5.4" width="0.254" layer="1"/>
 <wire x1="37" y1="16" x2="37.46" y2="16" width="0.254" layer="16"/>
 <wire x1="22.5" y1="12.5" x2="21" y2="11" width="0.254" layer="16"/>
@@
 <wire x1="4.5" y1="16" x2="4.44" y2="16" width="0.254" layer="16"/>
 <via x="31.5" y="7.5" extent="1-16" drill="0.6096"/>
+<contactref element="C1" pad="1"/>
+<wire x1="31.5" y1="6" x2="31.375" y2="5.75" width="0.1524" layer="1"/>
 </signal>
 <signal name="N$3">
-<contactref element="R25" pad="2"/>
+<contactref element="R2" pad="2"/>
 <contactref element="T1" pad="B"/>
 <wire x1="9.5" y1="6.5" x2="9.5" y2="3" width="0.254" layer="1"/>
@@
 </signal>
 <signal name="BACKLIGHT">
-<contactref element="R25" pad="1"/>
+<contactref element="R2" pad="1"/>
 <contactref element="Y" pad="8"/>
 <wire x1="17.5" y1="3" x2="11" y2="3" width="0.254" layer="1"/>
